File: pcb/stairshieldtoheaven.sch (KiCad schematic (older format))
At the start: 27 parts, among them P1 CONN_10X2, P10 5, P11 6, P12 7, P13 8, P14 9, P15 10, P16 11, P17 12, P18 13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

Commit message: massive rename improved version
Parts:
- added R1: RPLD, Resistors_ThroughHole:Resistor_Horizontal_RM10mm, symbol R
- added R2, R3: RL, Resistors_ThroughHole:Resistor_Horizontal_RM10mm, symbol R
Connections:
- wire segments 107 -> 109
Changed lines of the file:
@@
 LIBS:contrib
 LIBS:valves
-LIBS:crumpschemes
-LIBS:stairsheeldtoheaven-cache
+LIBS:stairshieldtoheaven-cache
 EELAYER 25 0
 EELAYER END
@@
 encoding utf-8
 Sheet 1 1
-Title "StairSheeldtoHeaven"
+Title "StairShieldtoHeaven"
 Date "07 oct. 2015"
 Rev "0.1"
@@
 	0    1    1    0
 $EndComp
-Text Label 4300 4250 3    60   ~ 0
+Text Label 4300 3800 3    60   ~ 0
 data
-Text Label 4100 4275 3    60   ~ 0
+Text Label 4100 3800 3    60   ~ 0
 clock
 Text Label 2650 3500 3    60   ~ 0
@@
 	1500 2300 1100 2300
 Connection ~ 1100 2300
-Wire Wire Line
-	4300 4500 4300 4250
 Wire Wire Line
 	2750 3500 2750 3650
@@
 Wire Wire Line
 	3400 1600 3550 1600
-Wire Wire Line
-	4100 4500 4100 4275
 $Comp
 L JUMPER JP2
@@
 Wire Wire Line
 	2150 4375 2150 4750
+$Comp
+L R R3
+U 1 1 5616E140
+P 4300 4250
+F 0 "R3" V 4380 4250 40  0000 C CNN
+F 1 "RL" V 4307 4251 40  0000 C CNN
+F 2 "Resistors_ThroughHole:Resistor_Horizontal_RM10mm" V 4230 4250 30  0001 C CNN
+F 3 "" H 4300 4250 30  0000 C CNN
+	1    4300 4250
+	1    0    0    -1
+$EndComp
+$Comp
+L R R2
+U 1 1 5616E395
+P 4100 4250
+F 0 "R2" V 4180 4250 40  0000 C CNN
+F 1 "RL" V 4107 4251 40  0000 C CNN
+F 2 "Resistors_ThroughHole:Resistor_Horizontal_RM10mm" V 4030 4250 30  0001 C CNN
+F 3 "" H 4100 4250 30  0000 C CNN
+	1    4100 4250
+	1    0    0    -1
+$EndComp
+$Comp
+L R R1
+U 1 1 5616E3F5
+P 3775 4500
+F 0 "R1" V 3855 4500 40  0000 C CNN
+F 1 "RPLD" V 3782 4501 40  0000 C CNN
+F 2 "Resistors_ThroughHole:Resistor_Horizontal_RM10mm" V 3705 4500 30  0001 C CNN
+F 3 "" H 3775 4500 30  0000 C CNN
+	1    3775 4500
+	0    1    1    0
+$EndComp
+Wire Wire Line
+	4025 4500 4100 4500
+$Comp
+L GND-RESCUE-atxpowerboard #PWR010
+U 1 1 5616E92F
+P 3525 4675
+F 0 "#PWR010" H 3525 4675 30  0001 C CNN
+F 1 "GND" H 3525 4605 30  0001 C CNN
+F 2 "" H 3525 4675 60  0000 C CNN
+F 3 "" H 3525 4675 60  0000 C CNN
+	1    3525 4675
+	1    0    0    -1
+$EndComp
+Wire Wire Line
+	3525 4500 3525 4675
+Wire Wire Line
+	4100 3800 4100 4000
+Wire Wire Line
+	4300 3800 4300 4000
 $EndSCHEMATC

Commit message: Fix bad commit: add missing files
Parts:
- removed JP2: JUMPER, Pin_Headers:Pin_Header_Straight_1x02, symbol JUMPER
- removed R3: RL, Resistors_ThroughHole:Resistor_Horizontal_RM10mm, symbol R
- added SPI1: CONN_02X03, Pin_Headers:Pin_Header_Straight_2x03, symbol CONN_02X03
- R1: value RPLD -> R; footprint Resistors_ThroughHole:Resistor_Horizontal_RM10mm -> Resistors_ThroughHole:Resistor_Horizontal_RM15mm
- R2: value RL -> R; footprint Resistors_ThroughHole:Resistor_Horizontal_RM10mm -> Resistors_ThroughHole:Resistor_Horizontal_RM15mm
Connections:
- net labels added: MISO, MOSI, Reset, SCK, VCC, Vcc
- net labels removed: clock, data
- wire segments 109 -> 123
- no-connect marks 11 -> 9
